File: Hardware/Dev_Board/main_mcu.kicad_sch (KiCad schematic)
At the start: 1 part, among them U1 AT90USB1287-AUR

Commit message: Added EEPROM documentation
Parts:
- added C1: 10u, symbol Device:C
- added C2, C3: 100n, symbol Device:C
- added C4: 1u, symbol Device:C
- added C5, C6: 40p, symbol Device:C
- added D1, D2, D3, D4: LED, LED_SMD:LED_0603_1608Metric, symbol Device:LED
- added R1, R2, R3, R4: 1k, Resistor_SMD:R_0603_1608Metric, symbol Device:R
- added Y1: FOXSDLF/080-20, CRYSTAL_HC49SDLF_FXT, symbol Dev_Board:FOXSDLF_080-20
Connections:
- net +3V3: now also U1.20 (RESET), C1.1, C2.1, C3.1
- net GND: now also U1.6 (UGnd), C1.2, C2.2, C3.2, C4.2, C5.2, C6.2, R1.2, R2.2, R3.2, R4.2
- net at U1.23 (XTAL2): now also C5.1, Y1.1
- net at U1.24 (XTAL1): now also C6.1, Y1.2
- net at U1.48 (PA3_(AD3)): now also D1.2 (A)
- net at U1.49 (PA2_(AD2)): now also D2.2 (A)
- net at U1.50 (PA1_(AD1)): now also D3.2 (A)
- net at U1.51 (PA0_(AD0)): now also D4.2 (A)
- net at U1.7 (UCap): now also C4.1
- new net: D1.1 (K), R1.1
- new net: D4.1 (K), R4.1
- new net: D2.1 (K), R2.1
- new net: D3.1 (K), R3.1
Other:
- note added: "8 MHz Oscillator"
- note added: "LED Bank"
- note added: "Power Supply"
