File: Hardware/Dev_Board/primary_mcu.kicad_sch (KiCad schematic)
At the start: 16 parts, among them U1 AT90USB1287-AUR, Y1 FOXSDLF/080-20

Commit message: Added the temperature sensor
Other:
- title: (none) -> Primary MCU
Changed lines of the file:
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@@
 	(paper "A4")
 	(title_block
+		(title "Primary MCU")
 		(company "Helena Hounds")
 	)
